File: PCB/v1PCB.kicad_pcb (KiCad board)
At the start: 2 copper layers, 370 x 125.1 mm, 223 parts, among them SW1 SW_PUSH, SW2 SW_PUSH, U1 STM32F072CBUx, U2 MCP1700-3302E_SOT23

Commit message: Added ground fills around USBC
Routing:
- added copper zone on B.Cu, net GND
- added copper zone on F.Cu, net GND
Other:
- board size 370 x 125.1 mm -> 369.9 x 125.4 mm
Changed lines of the file:
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@@
   (general
     (thickness 1.6)
-    (drawings 7)
+    (drawings 9)
     (tracks 1380)
     (zones 0)
@@
     )
   )
-  (gr_line (start 110.33125 100.0125) (end 110.3 225.107) (layer Edge.Cuts) (width 0.1))
-  (gr_line (start 480.28125 100.0125) (end 480.25 225.107) (layer Edge.Cuts) (width 0.2))
-  (gr_line (start 110.33125 100.0125) (end 480.28125 100.0125) (layer Edge.Cuts) (width 0.2))
-  (gr_line (start 480.25 225.107) (end 110.3 225.107) (layer Edge.Cuts) (width 0.2))
+  (gr_line (start 477.8375 225.425) (end 112.7125 225.425) (layer Edge.Cuts) (width 0.2))
+  (gr_line (start 480.21875 102.39375) (end 480.21875 223.04375) (layer Edge.Cuts) (width 0.2))
+  (gr_line (start 112.7125 100.0125) (end 477.8375 100.0125) (layer Edge.Cuts) (width 0.2))
+  (gr_line (start 110.33125 102.39375) (end 110.33125 223.04375) (layer Edge.Cuts) (width 0.2))
+  (gr_arc (start 477.8375 102.39375) (end 480.21875 102.39375) (angle -90) (layer Edge.Cuts) (width 0.2))
+  (gr_arc (start 477.8375 223.04375) (end 477.8375 225.425) (angle -90) (layer Edge.Cuts) (width 0.2))
+  (gr_arc (start 112.7125 223.04375) (end 110.33125 223.04375) (angle -90) (layer Edge.Cuts) (width 0.2))
+  (gr_arc (start 112.7125 102.39375) (end 112.7125 100.0125) (angle -90) (layer Edge.Cuts) (width 0.2))
   (gr_arc (start 113.475 175.03825) (end 113.475 175.03825) (angle -90) (layer Edge.Cuts) (width 0.2))
-  (gr_arc (start 480.25 225.107) (end 480.25 225.107) (angle -90) (layer Edge.Cuts) (width 0.2))
-  (gr_arc (start 110.3 225.107) (end 110.3 225.107) (angle 90) (layer Edge.Cuts) (width 0.2))
   (via (at 277.8125 219.075) (size 0.8) (drill 0.4) (layers F.Cu B.Cu) (net 1))
   (segment (start 277.01875 220.1775) (end 277.01875 219.86875) (width 0.3302) (layer B.Cu) (net 1))
@@
   (segment (start 135.89375 106.247) (end 135.89375 108.045462) (width 0.254) (layer B.Cu) (net 147))
   (segment (start 135.89375 108.045462) (end 137.195288 109.347) (width 0.254) (layer B.Cu) (net 147))
+  (zone (net 1) (net_name GND) (layer B.Cu) (hatch edge 0.508)
+    (connect_pads (clearance 0.508))
+    (min_thickness 0.254)
+    (fill yes (arc_segments 32) (thermal_gap 0.508) (thermal_bridge_width 0.508))
+    (polygon
+      (pts
+        (xy 141.2875 103.98125) (xy 127 103.98125) (xy 127 113.50625) (xy 141.2875 113.50625)
+      )
+    )
+  )
+  (zone (net 1) (net_name GND) (layer F.Cu) (hatch edge 0.508)
+    (connect_pads (clearance 0.508))
+    (min_thickness 0.254)
+    (fill yes (arc_segments 32) (thermal_gap 0.508) (thermal_bridge_width 0.508))
+    (polygon
+      (pts
+        (xy 141.2875 103.98125) (xy 127 103.98125) (xy 127 113.50625) (xy 141.2875 113.50625)
+      )
+    )
+  )
 )
