File: PCB/v1PCB.kicad_pcb (KiCad board)
At the start: 2 copper layers, 369.9 x 125.4 mm, 223 parts, among them SW1 SW_PUSH, SW2 SW_PUSH, U1 STM32F072CBUx, U2 MCP1700-3302E_SOT23

Commit message: Still need review, otherwise minor edits for the most part
Routing:
- net GND: track 451.1 -> 449.2 mm
Other:
- board text added: "ML JTM V1"
Changed lines of the file:
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@@
   (general
     (thickness 1.6)
-    (drawings 9)
+    (drawings 10)
     (tracks 1380)
     (zones 0)
@@
     )
   )
+  (gr_text "ML\nJTM\nV1" (at 355.854 208.534) (layer F.SilkS)
+    (effects (font (size 1 1) (thickness 0.15)))
+  )
   (gr_line (start 477.8375 225.425) (end 112.7125 225.425) (layer Edge.Cuts) (width 0.2))
   (gr_line (start 480.21875 102.39375) (end 480.21875 223.04375) (layer Edge.Cuts) (width 0.2))
@@
   (segment (start 285.1 219.075) (end 288.13125 216.04375) (width 0.3302) (layer B.Cu) (net 1))
   (segment (start 277.8125 219.075) (end 285.1 219.075) (width 0.3302) (layer B.Cu) (net 1))
-  (segment (start 125.8085 104.267) (end 125.8085 106.246962) (width 0.3302) (layer F.Cu) (net 1))
-  (segment (start 125.295538 106.3625) (end 115.8875 106.3625) (width 0.3302) (layer F.Cu) (net 1))
-  (segment (start 125.8085 106.246962) (end 125.411076 106.246962) (width 0.3302) (layer F.Cu) (net 1))
   (segment (start 115.8875 106.3625) (end 113.50625 108.74375) (width 0.3302) (layer F.Cu) (net 1))
   (segment (start 274.6375 219.86875) (end 276.71 219.86875) (width 0.3302) (layer B.Cu) (net 1))
   (segment (start 127.634038 219.86875) (end 274.6375 219.86875) (width 0.3302) (layer F.Cu) (net 1))
-  (segment (start 125.411076 106.246962) (end 125.295538 106.3625) (width 0.3302) (layer F.Cu) (net 1))
   (segment (start 276.71 219.86875) (end 277.01875 220.1775) (width 0.3302) (layer B.Cu) (net 1))
   (via (at 274.6375 219.86875) (size 0.8) (drill 0.4) (layers F.Cu B.Cu) (net 1))
@@
   (segment (start 138.1125 107.41575) (end 138.1125 109.5375) (width 0.3302) (layer B.Cu) (net 1))
   (via (at 128.778 109.601) (size 0.8) (drill 0.4) (layers F.Cu B.Cu) (net 1))
-  (segment (start 125.8085 106.6315) (end 125.8085 104.267) (width 0.3302) (layer F.Cu) (net 1))
   (segment (start 128.778 109.601) (end 125.8085 106.6315) (width 0.3302) (layer F.Cu) (net 1))
   (segment (start 129.2375 111.125) (end 129.2375 110.475) (width 0.3302) (layer B.Cu) (net 1))
@@
   (segment (start 130.91875 106.247) (end 130.91875 106.672) (width 0.3302) (layer B.Cu) (net 1))
   (segment (start 130.175 107.41575) (end 130.175 108.971815) (width 0.3302) (layer B.Cu) (net 1))
+  (segment (start 125.8085 106.6315) (end 125.8085 106.4745) (width 0.3302) (layer F.Cu) (net 1))
+  (segment (start 125.8085 106.4745) (end 125.8085 105.8695) (width 0.3302) (layer F.Cu) (net 1))
+  (segment (start 125.8085 105.8695) (end 125.8085 104.267) (width 0.3302) (layer F.Cu) (net 1))
+  (segment (start 125.5395 106.3625) (end 125.8085 106.6315) (width 0.381) (layer F.Cu) (net 1))
+  (segment (start 115.8875 106.3625) (end 125.5395 106.3625) (width 0.381) (layer F.Cu) (net 1))
   (segment (start 120.015 147.1295) (end 124.7775 151.892) (width 0.254) (layer F.Cu) (net 2))
   (segment (start 120.015 132.842) (end 120.015 147.1295) (width 0.254) (layer F.Cu) (net 2))

Commit message: Minor edits to cap values. Read previous comments
Parts:
- moved C1 2.29 mm to (305.5, 211.9)
- moved C10 2.29 mm to (292.8, 218.3)
- moved C2 2.29 mm to (307.1, 211.9)
- moved C3 2.29 mm to (296.8, 203.4)
- moved C4 2.29 mm to (294.4, 218.3)
- moved C6 2.29 mm to (300.1, 223.1)
- moved C7 2.29 mm to (296.8, 201.8)
- moved C8 2.29 mm to (300.1, 221.5)
- moved R1 2.29 mm to (302.3, 221.5)
- moved R2 2.29 mm to (290.4, 215.1)
- moved U1 2.29 mm to (299.1, 215.9)
Routing:
- net GND: track 449.2 -> 453.9 mm
- net +3V3: track 317.9 -> 322.0 mm
- net col10: track 131.5 -> 128.6 mm
- net col15: track 205.4 -> 203.0 mm
- net row1: track 601.9 -> 599.6 mm
- net col3: track 260.1 -> 262.4 mm
- net col0: track 280.7 -> 283.0 mm
- net col7: track 141.1 -> 143.4 mm
- net col4: track 212.4 -> 214.6 mm
- net col17: track 243.8 -> 241.5 mm
- net col13: track 174.6 -> 172.3 mm
- net col8: track 147.7 -> 149.9 mm
- net col5: track 171.6 -> 173.9 mm
- net col2: track 243.5 -> 245.8 mm
- net col18: track 257.8 -> 255.6 mm
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
Commit message: Added PCB cutouts, added CAD files for the case.
Routing:
- net +3V3: track 322.0 -> 319.1 mm
- net D+: track 291.2 -> 293.5 mm
- net D-: track 291.2 -> 292.8 mm
Other:
- outline, holes or cut-outs redrawn

Commit message: Redo all traces because MCU got moved to bottom. Continue refining CAD model.
Parts:
- C1, C2, C3, C4, C6, C7, C8, U1: moved to B.Cu
- K_32, K_54, K_87: footprint MX_Only:MXOnly-1U-NoLED -> MX_Only:MXOnly-2U-NoLED
- K_67, K_71, K_91: footprint MX_Only:MXOnly-1U-NoLED -> MX_Only:MXOnly-2.25U-NoLED
- K_82: footprint MX_Only:MXOnly-1U-NoLED -> MX_Only:MXOnly-1.75U-NoLED
- K_93: footprint MX_Only:MXOnly-1U-NoLED -> MX_Only:MXOnly-3U-NoLED
- moved R1 212.7 mm to (90.2, 206.4)
- moved R2 200.3 mm to (90.6, 201.9)
- moved C10 187.3 mm to (116.0, 156.4), turned to 0 degrees
- moved U2 177.8 mm to (116.0, 152.4), turned to 270 degrees
- moved C9 173.8 mm to (116.8, 153.2), turned to 0 degrees
- moved SW1 27.2 mm to (88.4, 186.8)
- moved SW2 27.2 mm to (88.4, 194.3)
- moved C2 22.9 mm to (284.5, 208.1)
- moved C1 19.8 mm to (286.1, 208.1)
- moved K_54 9.53 mm to (466.7, 164.0), turned to 270 degrees
- moved K_87 9.52 mm to (466.7, 202.1), turned to 270 degrees
- moved C6 9.50 mm to (291.4, 219.3), turned to 0 degrees
- moved C8 9.50 mm to (291.4, 217.7), turned to 0 degrees
- moved U1 7.73 mm to (292.4, 212.1)
- moved C7 6.78 mm to (301.5, 206.7), turned to 90 degrees
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Connections:
- U1 pad 10: row0 -> Net-(U1-Pad10)
- U1 pad 11: row1 -> Net-(U1-Pad11)
- U1 pad 12: row2 -> Net-(U1-Pad12)
- U1 pad 13: row3 -> Net-(U1-Pad13)
- U1 pad 14: row4 -> Net-(U1-Pad14)
- U1 pad 15: row5 -> Net-(U1-Pad15)
- U1 pad 16: col18 -> Net-(U1-Pad16)
- U1 pad 17: col17 -> Net-(U1-Pad17)
- U1 pad 18: col16 -> Net-(U1-Pad18)
- U1 pad 19: col15 -> Net-(U1-Pad19)
- U1 pad 20: col14 -> Net-(U1-Pad20)
- U1 pad 21: col13 -> Net-(U1-Pad21)
- U1 pad 22: col12 -> Net-(U1-Pad22)
- U1 pad 25: col11 -> Net-(U1-Pad25)
- U1 pad 26: col10 -> Net-(U1-Pad26)
- U1 pad 27: col9 -> Net-(U1-Pad27)
- U1 pad 28: col8 -> Net-(U1-Pad28)
- U1 pad 29: col7 -> Net-(U1-Pad29)
- U1 pad 30: col6 -> Net-(U1-Pad30)
- U1 pad 37: col5 -> Net-(U1-Pad37)
- U1 pad 38: col4 -> Net-(U1-Pad38)
- U1 pad 39: col3 -> Net-(U1-Pad39)
- U1 pad 40: col2 -> Net-(U1-Pad40)
- U1 pad 41: col1 -> Net-(U1-Pad41)
- U1 pad 42: col0 -> Net-(U1-Pad42)
Routing:
- net GND: track 453.9 -> 122.9 mm, vias 10 -> 3
- net +3V3: track 319.1 -> 12.2 mm, vias 8 -> 0
- net row0: track 621.7 -> 353.4 mm, vias 1 -> 0
- net col18: track 255.6 -> 0.00 mm
- net row1: track 599.6 -> 352.8 mm, vias 1 -> 0
- net +5V: track 288.3 -> 54.4 mm
- net NRST: track 231.2 -> 0.54 mm, vias 1 -> 0
- net row2: track 568.9 -> 344.3 mm, vias 1 -> 0
- net row3: track 549.2 -> 326.5 mm, vias 1 -> 0
- net BOOT0: track 203.0 -> 0.00 mm, vias 1 -> 0
- net row4: track 524.3 -> 342.0 mm, vias 1 -> 0
- net col0: track 283.0 -> 104.1 mm
- net col2: track 245.8 -> 86.1 mm
- net col1: track 267.8 -> 112.9 mm
- net row5: track 494.7 -> 345.0 mm, vias 1 -> 0
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- removed copper zone on B.Cu, net GND
- removed copper zone on F.Cu, net GND

Commit message: Finished relocating MCU, prep for review. Need to adjust cutouts for case mounting.
Parts:
- moved R1 40.7 mm to (114.0, 173.4), turned to 270 degrees
- moved R2 30.1 mm to (119.3, 192.9)
- moved SW1 28.4 mm to (116.0, 179.8)
- moved SW2 28.4 mm to (116.0, 187.3)
- moved C3 2.50 mm to (297.6, 207.7)
- moved C7 2.50 mm to (299.2, 207.7)
- moved C1 1.55 mm to (287.3, 209.0)
- moved C2 1.55 mm to (285.8, 209.0)
- moved C4 0.78 mm to (297.3, 215.2)
Connections:
- U1 pad 2: Net-(U1-Pad2) -> row4
- U1 pad 20: Net-(U1-Pad20) -> col0
- U1 pad 21: Net-(U1-Pad21) -> col1
- U1 pad 22: Net-(U1-Pad22) -> col2
- U1 pad 25: Net-(U1-Pad25) -> col3
- U1 pad 26: Net-(U1-Pad26) -> col4
- U1 pad 27: Net-(U1-Pad27) -> col5
- U1 pad 28: Net-(U1-Pad28) -> col6
- U1 pad 29: Net-(U1-Pad29) -> col7
- U1 pad 3: Net-(U1-Pad3) -> row3
- U1 pad 30: Net-(U1-Pad30) -> col8
- U1 pad 31: Net-(U1-Pad31) -> col9
- U1 pad 34: Net-(U1-Pad34) -> col10
- U1 pad 37: Net-(U1-Pad37) -> col11
- U1 pad 38: Net-(U1-Pad38) -> col12
- U1 pad 39: Net-(U1-Pad39) -> col13
- U1 pad 4: Net-(U1-Pad4) -> row2
- U1 pad 40: Net-(U1-Pad40) -> col14
- U1 pad 41: Net-(U1-Pad41) -> col15
- U1 pad 42: Net-(U1-Pad42) -> col16
- U1 pad 43: Net-(U1-Pad43) -> col17
- U1 pad 45: Net-(U1-Pad45) -> col18
- U1 pad 46: Net-(U1-Pad46) -> row5
- U1 pad 5: Net-(U1-Pad5) -> row1
- U1 pad 6: Net-(U1-Pad6) -> row0
Routing:
- net NRST: track 0.54 -> 321.9 mm, vias 0 -> 1
- net +3V3: track 12.2 -> 329.6 mm, vias 0 -> 8
- net GND: track 122.9 -> 436.6 mm, vias 3 -> 8
- net row0: track 353.4 -> 650.6 mm
- net col18: track 0.00 -> 280.8 mm, vias 0 -> 1
- net row1: track 352.8 -> 629.3 mm
- net row3: track 326.5 -> 577.1 mm
- net row2: track 344.3 -> 594.6 mm
- net BOOT0: track 0.00 -> 239.3 mm, vias 0 -> 2
- net row4: track 342.0 -> 552.1 mm
- net row5: track 345.0 -> 553.0 mm
- net col0: track 104.1 -> 278.2 mm, vias 0 -> 1
- net col17: track 95.2 -> 252.7 mm, vias 0 -> 1
- net col2: track 86.1 -> 239.8 mm, vias 0 -> 1
- net col1: track 112.9 -> 261.8 mm, vias 0 -> 1
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Other:
- outline, holes or cut-outs redrawn
- net class Power: trace_width 0.381 -> 0.3302

Commit message: added GND fill
Routing:
- added copper zone on B.Cu, net GND
- added copper zone on F.Cu, net GND
Other:
- outline, holes or cut-outs redrawn
Changed lines of the file:
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@@
   (general
     (thickness 1.6)
-    (drawings 16)
+    (drawings 10)
     (tracks 1499)
     (zones 0)
@@
     )
   )
+  (gr_line (start 112.7125 100.0125) (end 477.8375 100.0125) (layer Edge.Cuts) (width 0.2))
   (gr_line (start 112.7125 225.425) (end 477.8375 225.425) (layer Edge.Cuts) (width 0.2))
-  (gr_line (start 416.71875 100.0125) (end 477.8375 100.0125) (layer Edge.Cuts) (width 0.2))
-  (gr_line (start 297.65625 100.0125) (end 408.78125 100.0125) (layer Edge.Cuts) (width 0.2))
-  (gr_line (start 202.40625 100.0125) (end 289.71875 100.0125) (layer Edge.Cuts) (width 0.2))
-  (gr_line (start 112.7125 100.0125) (end 194.46875 100.0125) (layer Edge.Cuts) (width 0.1))
-  (gr_arc (start 198.4375 100.0125) (end 194.46875 100.0125) (angle -180) (layer Edge.Cuts) (width 0.1))
-  (gr_arc (start 412.75 100.0125) (end 408.78125 100.0125) (angle -180) (layer Edge.Cuts) (width 0.2))
-  (gr_arc (start 293.6875 100.0125) (end 289.71875 100.0125) (angle -180) (layer Edge.Cuts) (width 0.2))
   (gr_text "ML\nJTM\nV1" (at 355.854 208.534) (layer F.SilkS)
     (effects (font (size 1 1) (thickness 0.15)))
@@
   (segment (start 135.89375 106.247) (end 135.89375 108.045462) (width 0.254) (layer B.Cu) (net 139))
   (segment (start 135.89375 108.045462) (end 137.195288 109.347) (width 0.254) (layer B.Cu) (net 139))
+  (zone (net 1) (net_name GND) (layer F.Cu) (hatch edge 0.508)
+    (connect_pads (clearance 0.508))
+    (min_thickness 0.254)
+    (fill yes (arc_segments 32) (thermal_gap 0.508) (thermal_bridge_width 0.508))
+    (polygon
+      (pts
+        (xy 140.97 105.41) (xy 128.27 105.41) (xy 128.27 113.03) (xy 140.97 113.03)
+      )
+    )
+  )
+  (zone (net 1) (net_name GND) (layer B.Cu) (hatch edge 0.508)
+    (connect_pads (clearance 0.508))
+    (min_thickness 0.254)
+    (fill yes (arc_segments 32) (thermal_gap 0.508) (thermal_bridge_width 0.508))
+    (polygon
+      (pts
+        (xy 140.97 105.41) (xy 128.27 105.41) (xy 128.27 113.03) (xy 140.97 113.03)
+      )
+    )
+  )
 )

Commit message: Rerouted some traces near stab holes
Parts:
- moved C3 2.95 mm to (300.5, 207.3)
- moved C7 2.95 mm to (302.1, 207.3)
- moved C4 1.53 mm to (298.8, 215.1)
Routing:
- net +3V3: track 329.6 -> 342.0 mm
- net row1: track 629.3 -> 637.8 mm
- net GND: track 436.6 -> 442.5 mm
- net row0: track 650.6 -> 654.0 mm
- net col10: track 142.3 -> 143.4 mm

Commit message: Fixed cutouts.
Routing:
- net NRST: track 321.9 -> 324.5 mm
- net +3V3: track 342.0 -> 343.9 mm
- net GND: track 442.5 -> 444.5 mm
Other:
- outline, holes or cut-outs redrawn
Changed lines of the file:
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@@
   (general
     (thickness 1.6)
-    (drawings 10)
-    (tracks 1515)
+    (drawings 20)
+    (tracks 1526)
     (zones 0)
     (modules 223)
@@
     )
   )
-  (gr_line (start 112.7125 100.0125) (end 477.8375 100.0125) (layer Edge.Cuts) (width 0.2))
-  (gr_line (start 112.7125 225.425) (end 477.8375 225.425) (layer Edge.Cuts) (width 0.2))
+  (gr_line (start 199.23125 225.425) (end 112.7125 225.425) (layer Edge.Cuts) (width 0.2))
+  (gr_line (start 384.175 225.425) (end 205.58125 225.425) (layer Edge.Cuts) (width 0.2))
+  (gr_line (start 477.8375 225.425) (end 390.525 225.425) (layer Edge.Cuts) (width 0.2))
+  (gr_line (start 390.525 100.0125) (end 477.8375 100.0125) (layer Edge.Cuts) (width 0.2))
+  (gr_line (start 298.45 100.0125) (end 384.175 100.0125) (layer Edge.Cuts) (width 0.2))
+  (gr_line (start 205.58125 100.0125) (end 292.1 100.0125) (layer Edge.Cuts) (width 0.2))
+  (gr_line (start 112.7125 100.0125) (end 199.23125 100.0125) (layer Edge.Cuts) (width 0.2))
+  (gr_arc (start 387.35 100.0125) (end 384.175 100.0125) (angle -180) (layer Edge.Cuts) (width 0.2))
+  (gr_arc (start 295.275 100.0125) (end 292.1 100.0125) (angle -180) (layer Edge.Cuts) (width 0.2))
+  (gr_arc (start 202.40625 100.0125) (end 199.23125 100.0125) (angle -180) (layer Edge.Cuts) (width 0.2))
+  (gr_arc (start 387.35 225.425) (end 390.525 225.425) (angle -180) (layer Edge.Cuts) (width 0.2))
+  (gr_arc (start 202.40625 225.425) (end 205.58125 225.425) (angle -180) (layer Edge.Cuts) (width 0.2))
   (gr_text "ML\nJTM\nV1" (at 355.854 208.534) (layer F.SilkS)
     (effects (font (size 1 1) (thickness 0.15)))
@@
   (segment (start 292.22075 219.2655) (end 290.82375 220.6625) (width 0.3302) (layer B.Cu) (net 1))
   (segment (start 290.82375 220.6625) (end 284.1625 220.6625) (width 0.3302) (layer B.Cu) (net 1))
-  (segment (start 129.904901 222.196001) (end 276.278999 222.196001) (width 0.3302) (layer F.Cu) (net 1))
-  (segment (start 116.4995 208.7906) (end 129.904901 222.196001) (width 0.3302) (layer F.Cu) (net 1))
-  (segment (start 276.278999 222.196001) (end 277.8125 220.6625) (width 0.3302) (layer F.Cu) (net 1))
-  (segment (start 277.8125 220.6625) (end 278.60625 219.86875) (width 0.3302) (layer F.Cu) (net 1))
   (segment (start 281.78125 219.86875) (end 282.575 220.6625) (width 0.3302) (layer F.Cu) (net 1))
   (segment (start 280.9875 219.86875) (end 281.78125 219.86875) (width 0.3302) (layer F.Cu) (net 1))
-  (segment (start 278.60625 219.86875) (end 280.9875 219.86875) (width 0.3302) (layer F.Cu) (net 1))
   (segment (start 283.36875 219.86875) (end 284.1625 220.6625) (width 0.3302) (layer F.Cu) (net 1))
   (segment (start 280.9875 219.86875) (end 283.36875 219.86875) (width 0.3302) (layer F.Cu) (net 1))
@@
   (segment (start 116.4995 178.6485) (end 116.4995 179.4105) (width 0.3302) (layer F.Cu) (net 1))
   (segment (start 116.4995 192.8265) (end 116.4995 198.4145) (width 0.3302) (layer F.Cu) (net 1))
-  (segment (start 116.4995 198.4145) (end 116.4995 208.7906) (width 0.3302) (layer F.Cu) (net 1))
   (segment (start 116.4995 198.3335) (end 116.4995 198.4145) (width 0.3302) (layer F.Cu) (net 1))
   (segment (start 119.253 195.58) (end 116.4995 198.3335) (width 0.3302) (layer F.Cu) (net 1))
@@
   (segment (start 295.527227 207.250541) (end 294.6675 208.110268) (width 0.3302) (layer B.Cu) (net 1))
   (segment (start 299.68571 207.25054) (end 295.527227 207.250541) (width 0.3302) (layer B.Cu) (net 1))
+  (segment (start 278.60625 219.86875) (end 280.9875 219.86875) (width 0.3302) (layer F.Cu) (net 1))
+  (segment (start 276.278999 222.196001) (end 278.60625 219.86875) (width 0.3302) (layer F.Cu) (net 1))
+  (segment (start 207.114751 222.196001) (end 276.278999 222.196001) (width 0.3302) (layer F.Cu) (net 1))
+  (segment (start 116.4995 198.4145) (end 116.4995 208.7906) (width 0.3302) (layer F.Cu) (net 1))
+  (segment (start 116.4995 208.7906) (end 129.904901 222.196001) (width 0.3302) (layer F.Cu) (net 1))
+  (segment (start 129.904901 222.196001) (end 197.697749 222.196001) (width 0.3302) (layer F.Cu) (net 1))
+  (segment (start 197.697749 222.196001) (end 200.025 219.86875) (width 0.3302) (layer F.Cu) (net 1))
+  (segment (start 200.025 219.86875) (end 204.7875 219.86875) (width 0.3302) (layer F.Cu) (net 1))
+  (segment (start 204.7875 219.86875) (end 207.114751 222.196001) (width 0.3302) (layer F.Cu) (net 1))
   (segment (start 120.015 147.1295) (end 124.7775 151.892) (width 0.254) (layer F.Cu) (net 2))
   (segment (start 120.015 132.842) (end 120.015 147.1295) (width 0.254) (layer F.Cu) (net 2))
@@
   (segment (start 290.64575 219.2655) (end 284.42715 219.2655) (width 0.3302) (layer B.Cu) (net 129))
   (segment (start 284.42715 219.2655) (end 283.397399 220.295251) (width 0.3302) (layer B.Cu) (net 129))
-  (segment (start 129.685281 222.726211) (end 277.336289 222.726211) (width 0.3302) (layer F.Cu) (net 129))
-  (segment (start 115.5295 208.57043) (end 129.685281 222.726211) (width 0.3302) (layer F.Cu) (net 129))
-  (segment (start 277.336289 222.726211) (end 277.653828 223.04375) (width 0.3302) (layer F.Cu) (net 129))
   (segment (start 281.78125 223.04375) (end 282.575 222.25) (width 0.3302) (layer F.Cu) (net 129))
-  (segment (start 277.653828 223.04375) (end 281.78125 223.04375) (width 0.3302) (layer F.Cu) (net 129))
   (segment (start 283.36875 223.04375) (end 284.1625 222.25) (width 0.3302) (layer F.Cu) (net 129))
   (segment (start 282.575 223.04375) (end 283.36875 223.04375) (width 0.3302) (layer F.Cu) (net 129))
   (segment (start 281.78125 223.04375) (end 282.575 223.04375) (width 0.3302) (layer F.Cu) (net 129))
-  (segment (start 115.5295 187.8735) (end 115.5295 208.57043) (width 0.3302) (layer F.Cu) (net 129))
   (segment (start 113.630999 185.974999) (end 115.5295 187.8735) (width 0.3302) (layer F.Cu) (net 129))
   (segment (start 113.600999 185.974999) (end 113.630999 185.974999) (width 0.3302) (layer F.Cu) (net 129))
@@
   (segment (start 293.932337 220.865305) (end 293.932337 218.742673) (width 0.3302) (layer F.Cu) (net 129))
   (segment (start 293.382013 221.415629) (end 293.932337 220.865305) (width 0.3302) (layer F.Cu) (net 129))
+  (segment (start 277.653828 223.04375) (end 281.78125 223.04375) (width 0.3302) (layer F.Cu) (net 129))
+  (segment (start 206.895131 222.726211) (end 277.336289 222.726211) (width 0.3302) (layer F.Cu) (net 129))
+  (segment (start 115.5295 187.8735) (end 115.5295 208.57043) (width 0.3302) (layer F.Cu) (net 129))
+  (segment (start 115.5295 208.57043) (end 129.685281 222.726211) (width 0.3302) (layer F.Cu) (net 129))
+  (segment (start 277.336289 222.726211) (end 277.653828 223.04375) (width 0.3302) (layer F.Cu) (net 129))
+  (segment (start 129.685281 222.726211) (end 197.917369 222.726211) (width 0.3302) (layer F.Cu) (net 129))
+  (segment (start 197.917369 222.726211) (end 200.24462 220.39896) (width 0.3302) (layer F.Cu) (net 129))
+  (segment (start 200.24462 220.39896) (end 204.56788 220.39896) (width 0.3302) (layer F.Cu) (net 129))
+  (segment (start 204.56788 220.39896) (end 206.895131 222.726211) (width 0.3302) (layer F.Cu) (net 129))
   (via (at 293.167236 220.438964) (size 0.8) (drill 0.4) (layers F.Cu B.Cu) (net 130))
   (segment (start 293.167236 217.935926) (end 293.167236 220.438964) (width 0.254) (layer B.Cu) (net 130))
@@
   (segment (start 290.629199 222.977001) (end 292.767237 220.838963) (width 0.254) (layer B.Cu) (net 130))
   (segment (start 117.39798 210.274759) (end 130.100222 222.977001) (width 0.254) (layer B.Cu) (net 130))
-  (segment (start 130.100222 222.977001) (end 290.629199 222.977001) (width 0.254) (layer B.Cu) (net 130))
   (segment (start 117.39798 189.562058) (end 117.39798 210.274759) (width 0.254) (layer B.Cu) (net 130))
   (segment (start 118.612039 188.347999) (end 117.39798 189.562058) (width 0.254) (layer B.Cu) (net 130))
@@
   (segment (start 125.766813 214.443601) (end 121.703211 210.379999) (width 0.254) (layer B.Cu) (net 130))
   (segment (start 114.046 176.237) (end 138.817148 176.237) (width 0.254) (layer B.Cu) (net 130))
+  (segment (start 196.916749 222.977001) (end 200.025 219.86875) (width 0.254) (layer B.Cu) (net 130))
+  (segment (start 130.100222 222.977001) (end 196.916749 222.977001) (width 0.254) (layer B.Cu) (net 130))
+  (segment (start 200.025 219.86875) (end 204.7875 219.86875) (width 0.254) (layer B.Cu) (net 130))
+  (segment (start 204.7875 219.86875) (end 207.895751 222.977001) (width 0.254) (layer B.Cu) (net 130))
+  (segment (start 207.895751 222.977001) (end 290.629199 222.977001) (width 0.254) (layer B.Cu) (net 130))
   (via (at 306.668032 213.283329) (size 0.8) (drill 0.4) (layers F.Cu B.Cu) (net 131))
   (segment (start 295.855 212.84) (end 306.224703 212.84) (width 0.254) (layer B.Cu) (net 131))
