File: PCB/_autosave-v1PCB.kicad_pcb (KiCad board)
At the start: 2 copper layers, 369.9 x 125.4 mm, 223 parts, among them SW1 SW_PUSH, SW2 SW_PUSH, U1 STM32F072CBUx, U2 MCP1700-3302E_SOT23

Commit message: Moved MCU so that stabs won't interfere. Almost cried.
Parts:
- moved C1 2.29 mm to (305.5, 211.9)
- moved C10 2.29 mm to (292.8, 218.3)
- moved C2 2.29 mm to (307.1, 211.9)
- moved C3 2.29 mm to (296.8, 203.4)
- moved C4 2.29 mm to (294.4, 218.3)
- moved C6 2.29 mm to (300.1, 223.1)
- moved C7 2.29 mm to (296.8, 201.8)
- moved C8 2.29 mm to (300.1, 221.5)
- moved R1 2.29 mm to (302.3, 221.5)
- moved R2 2.29 mm to (290.4, 215.1)
- moved U1 2.29 mm to (299.1, 215.9)
Routing:
- net +3V3: track 317.9 -> 160.2 mm
- net col10: track 131.5 -> 128.6 mm
- net GND: track 451.1 -> 453.9 mm
- net col15: track 205.4 -> 203.0 mm
- net row1: track 601.9 -> 599.6 mm
- net col3: track 260.1 -> 262.4 mm
- net col0: track 280.7 -> 283.0 mm
- net col7: track 141.1 -> 143.4 mm
- net col4: track 212.4 -> 214.6 mm
- net col17: track 243.8 -> 241.5 mm
- net col13: track 174.6 -> 172.3 mm
- net col8: track 147.7 -> 149.9 mm
- net col5: track 171.6 -> 173.9 mm
- net col2: track 243.5 -> 245.8 mm
- net col18: track 257.8 -> 255.6 mm
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- added copper zone on B.Cu, net GND
- added copper zone on F.Cu, net GND
Other:
- board text added: "ML JTM V1"

Commit message: Reorganizing
Routing:
- net +3V3: track 160.2 -> 322.0 mm
Changed lines of the file:
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@@
     (thickness 1.6)
     (drawings 10)
-    (tracks 1385)
+    (tracks 1388)
     (zones 0)
     (modules 223)
@@
   (segment (start 287.401 221.869) (end 285.115 221.869) (width 0.381) (layer F.Cu) (net 129))
   (segment (start 285.2025 224.63125) (end 282.9165 224.63125) (width 0.381) (layer F.Cu) (net 129))
+  (segment (start 193.480625 223.841375) (end 282.126625 223.841375) (width 0.381) (layer F.Cu) (net 129))
+  (segment (start 192.69075 224.63125) (end 193.480625 223.841375) (width 0.381) (layer F.Cu) (net 129))
+  (segment (start 120.648381 224.63125) (end 192.69075 224.63125) (width 0.381) (layer F.Cu) (net 129))
   (via (at 297.561 222.25) (size 0.8) (drill 0.4) (layers F.Cu B.Cu) (net 130))
   (segment (start 297.561 221.7125) (end 297.561 222.25) (width 0.254) (layer F.Cu) (net 130))
