File: PCB/Plate/Plate/Plate.kicad_pcb (KiCad board)
At the start: 2 copper layers, 380 x 127.9 mm, 10 parts

Commit message: Updates
Parts:
- R1: moved to B.Cu
- moved R1 4.27 mm to (273.1, 168.3)
Routing:
- net (no net): track 6.91 -> 0.00 mm
Other:
- outline, holes or cut-outs redrawn
- board text added: "ML JTM V1.1"

Commit message: Updates to PCB and CAD. Incorrect PaP files, beware EasyEDA
Parts:
- removed H1, H2, H3, H4, H5, H6, H7, H8, H9: MountingHole, MountingHole:MountingHole_2.1mm
- R1: moved to F.Cu
- moved R1 3.28 mm to (273.1, 171.6), turned to 180 degrees
Other:
- outline, holes or cut-outs redrawn
