File: PCB/Plate/Plate/Plate.sch (KiCad schematic (older format))
At the start: 10 parts

Commit message: Updates to PCB and CAD. Incorrect PaP files, beware EasyEDA
Parts:
- removed H1, H2, H3, H4, H5, H6, H7, H8, H9: MountingHole, MountingHole:MountingHole_2.1mm, symbol Mechanical:MountingHole
- R1: symbol Device:R_Small -> Plate-rescue:R_Small-Device
Changed lines of the file:
@@
 EESchema Schematic File Version 4
-LIBS:Plate-cache
 EELAYER 30 0
 EELAYER END
@@
 $EndDescr
 $Comp
-L Device:R_Small R1
+L Plate-rescue:R_Small-Device R1
 U 1 1 5F2861F8
 P 4850 2700
@@
 	1    0    0    -1
 $EndComp
-$Comp
-L Mechanical:MountingHole H5
-U 1 1 5F3605E4
-P 3500 1300
-F 0 "H5" H 3600 1346 50  0000 L CNN
-F 1 "MountingHole" H 3600 1255 50  0000 L CNN
-F 2 "MountingHole:MountingHole_2.1mm" H 3500 1300 50  0001 C CNN
-F 3 "~" H 3500 1300 50  0001 C CNN
-	1    3500 1300
-	1    0    0    -1
-$EndComp
-$Comp
-L Mechanical:MountingHole H6
-U 1 1 5F360AF0
-P 3500 1900
-F 0 "H6" H 3600 1946 50  0000 L CNN
-F 1 "MountingHole" H 3600 1855 50  0000 L CNN
-F 2 "MountingHole:MountingHole_2.1mm" H 3500 1900 50  0001 C CNN
-F 3 "~" H 3500 1900 50  0001 C CNN
-	1    3500 1900
-	1    0    0    -1
-$EndComp
-$Comp
-L Mechanical:MountingHole H4
-U 1 1 5F360D38
-P 3450 2750
-F 0 "H4" H 3550 2796 50  0000 L CNN
-F 1 "MountingHole" H 3550 2705 50  0000 L CNN
-F 2 "MountingHole:MountingHole_2.1mm" H 3450 2750 50  0001 C CNN
-F 3 "~" H 3450 2750 50  0001 C CNN
-	1    3450 2750
-	1    0    0    -1
-$EndComp
-$Comp
-L Mechanical:MountingHole H9
-U 1 1 5F360EE4
-P 4800 1900
-F 0 "H9" H 4900 1946 50  0000 L CNN
-F 1 "MountingHole" H 4900 1855 50  0000 L CNN
-F 2 "MountingHole:MountingHole_2.1mm" H 4800 1900 50  0001 C CNN
-F 3 "~" H 4800 1900 50  0001 C CNN
-	1    4800 1900
-	1    0    0    -1
-$EndComp
-$Comp
-L Mechanical:MountingHole H7
-U 1 1 5F3610F0
-P 3950 2400
-F 0 "H7" H 4050 2446 50  0000 L CNN
-F 1 "MountingHole" H 4050 2355 50  0000 L CNN
-F 2 "MountingHole:MountingHole_2.1mm" H 3950 2400 50  0001 C CNN
-F 3 "~" H 3950 2400 50  0001 C CNN
-	1    3950 2400
-	1    0    0    -1
-$EndComp
-$Comp
-L Mechanical:MountingHole H8
-U 1 1 5F361326
-P 4500 1400
-F 0 "H8" H 4600 1446 50  0000 L CNN
-F 1 "MountingHole" H 4600 1355 50  0000 L CNN
-F 2 "MountingHole:MountingHole_2.1mm" H 4500 1400 50  0001 C CNN
-F 3 "~" H 4500 1400 50  0001 C CNN
-	1    4500 1400
-	1    0    0    -1
-$EndComp
-$Comp
-L Mechanical:MountingHole H2
-U 1 1 5F3615CC
-P 3100 1600
-F 0 "H2" H 3200 1646 50  0000 L CNN
-F 1 "MountingHole" H 3200 1555 50  0000 L CNN
-F 2 "MountingHole:MountingHole_2.1mm" H 3100 1600 50  0001 C CNN
-F 3 "~" H 3100 1600 50  0001 C CNN
-	1    3100 1600
-	1    0    0    -1
-$EndComp
-$Comp
-L Mechanical:MountingHole H1
-U 1 1 5F3617FC
-P 2950 2000
-F 0 "H1" H 3050 2046 50  0000 L CNN
-F 1 "MountingHole" H 3050 1955 50  0000 L CNN
-F 2 "MountingHole:MountingHole_2.1mm" H 2950 2000 50  0001 C CNN
-F 3 "~" H 2950 2000 50  0001 C CNN
-	1    2950 2000
-	1    0    0    -1
-$EndComp
-$Comp
-L Mechanical:MountingHole H3
-U 1 1 5F361A98
-P 3200 2300
-F 0 "H3" H 3300 2346 50  0000 L CNN
-F 1 "MountingHole" H 3300 2255 50  0000 L CNN
-F 2 "MountingHole:MountingHole_2.1mm" H 3200 2300 50  0001 C CNN
-F 3 "~" H 3200 2300 50  0001 C CNN
-	1    3200 2300
-	1    0    0    -1
-$EndComp
